File: rp2040_devboard.kicad_pcb (KiCad board)
At the start: 2 copper layers, 21 x 51 mm, 33 parts, among them J1 USB_C_Receptacle_USB2.0_14P, J2 Conn_01x20, J3 Conn_01x20, J4 Conn_01x03, SW1 SW_Push, U1 RP2040, U2 MCP1700x-330xxMB, U3 W25Q128JVS, Y1 Crystal_GND24

Commit message: routing and copper fill
Routing:
- net +3V3: track 14.4 -> 29.7 mm
- net (no net): track 0.00 -> 11.0 mm, vias 0 -> 2
- net +1V1: track 0.00 -> 3.01 mm
- net Net-(C16-Pad1): track 0.00 -> 2.10 mm
- net XIN: track 0.00 -> 1.66 mm
- added copper zone on F.Cu, net GND

Commit message: added a lot of tracing and routing and stuff i dont undersand anything though
Parts:
- moved R3 69.1 mm to (100.5, 35.3)
- moved R4 65.6 mm to (100.5, 47.5)
- moved R5 61.7 mm to (99.2, 63.4)
- moved SW1 52.2 mm to (96.0, 67.0), turned to 180 degrees
- moved J2 18.0 mm to (88.0, 28.5)
- moved J3 18.0 mm to (106.0, 28.5)
- moved R1 2.30 mm to (98.5, 35.3)
- moved R2 1.99 mm to (96.5, 35.3)
- moved R7 0.75 mm to (96.5, 59.5)
Routing:
- net GPIO0: track 0.00 -> 28.0 mm
- net GPIO1: track 0.00 -> 24.3 mm
- net GPIO29_ADC3: track 0.00 -> 23.5 mm
- net GPIO16: track 0.00 -> 22.8 mm
- net GPIO15: track 0.00 -> 22.0 mm
- net GPIO17: track 0.00 -> 20.4 mm
- net SWCLK: track 0.00 -> 20.0 mm
- net GPIO2: track 0.00 -> 19.6 mm
- net GPIO14: track 0.00 -> 19.4 mm, vias 0 -> 1
- net GPIO28_ADC2: track 0.00 -> 19.2 mm
- net SWD: track 0.00 -> 19.1 mm
- net GPIO3: track 0.00 -> 17.5 mm
- net GPIO27_ADC1: track 0.00 -> 16.7 mm
- net GPIO18: track 0.00 -> 16.1 mm
- net GPIO13: track 0.00 -> 15.6 mm
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- added copper zone on B.Cu, net GND
Other:
- board size 21 x 51 mm -> 21 x 52 mm

Commit message: so i was told my routing was trash. i'll redo it!
Parts:
- C13, C14: footprint Capacitor_SMD:C_0201_0603Metric -> Capacitor_SMD:C_0603_1608Metric
- moved C7 18.0 mm to (119.5, 54.0)
- moved C8 16.2 mm to (118.0, 52.5), turned to 0 degrees
- moved C9 15.4 mm to (117.5, 56.5)
- moved C3 12.7 mm to (103.5, 37.5)
- moved C1 12.5 mm to (114.5, 53.5)
- moved C4 11.9 mm to (101.5, 37.5)
- moved C2 11.4 mm to (99.0, 38.0)
- moved C6 11.0 mm to (113.0, 56.0)
- moved C5 7.52 mm to (101.5, 42.0), turned to 0 degrees
- moved C12 4.76 mm to (102.5, 48.5)
- moved R3 3.09 mm to (97.5, 36.0), turned to -90 degrees
- moved C14 2.39 mm to (98.3, 40.5)
- moved R5 1.40 mm to (100.5, 64.0)
- moved U2 1.35 mm to (94.5, 39.5)
- moved C13 0.88 mm to (93.8, 36.0)
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Routing:
- net VBUS: track 17.3 -> 7.52 mm
- net +3V3: track 28.2 -> 33.7 mm
- net Net-(C16-Pad1): track 2.18 -> 0.24 mm
- net Net-(J1-CC1): track 1.86 -> 0.00 mm
- net RUN: track 11.7 -> 13.5 mm
- net XIN: track 1.66 -> 0.00 mm
- net Net-(R7-Pad1): track 11.7 -> 12.8 mm
- net GPIO17: track 20.4 -> 21.3 mm
- net GPIO14: track 19.4 -> 20.2 mm, vias 1 -> 0
- net GPIO16: track 22.8 -> 22.2 mm
- net GPIO10: track 9.25 -> 9.82 mm
- net GND: track 0.00 -> 0.12 mm, vias 31 -> 28
- removed copper zone on B.Cu, net GND
- removed copper zone on F.Cu, net GND
Other:
- board size 21 x 52 mm -> 21.9 x 52.6 mm

Commit message: i think i've routed this at least 5 times over at this point
Parts:
- moved C3 34.7 mm to (99.3, 72.0), turned to -90 degrees
- moved C2 34.0 mm to (98.3, 72.0), turned to -90 degrees
- moved C13 30.8 mm to (99.8, 66.2), turned to 90 degrees
- moved C14 28.8 mm to (99.8, 69.3), turned to 90 degrees
- moved U2 28.3 mm to (96.4, 67.8)
- moved C1 25.6 mm to (96.8, 71.9), turned to -90 degrees
- moved SW1 25.3 mm to (96.5, 41.7), turned to -90 degrees
- moved C9 24.7 mm to (103.0, 36.5), turned to 180 degrees
- moved C7 22.6 mm to (103.0, 38.5)
- moved C8 21.2 mm to (103.0, 37.5), turned to 180 degrees
- moved C6 19.3 mm to (103.0, 39.5), turned to 180 degrees
- moved C4 17.9 mm to (101.5, 55.4), turned to 0 degrees
- moved R6 15.4 mm to (95.0, 45.3), turned to 180 degrees
- moved R7 15.1 mm to (93.5, 44.8), turned to -90 degrees
- moved R3 12.1 mm to (100.5, 47.8)
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Routing:
- net +1V1: track 3.01 -> 19.8 mm
- net USB_D+: track 2.78 -> 19.3 mm
- net VBUS: track 7.52 -> 22.1 mm
- net +3V3: track 33.7 -> 48.2 mm
- net RUN: track 13.5 -> 0.00 mm, vias 1 -> 0
- net (no net): track 11.0 -> 0.00 mm, vias 2 -> 3
- net Net-(R7-Pad1): track 12.8 -> 3.20 mm
- net Net-(C16-Pad1): track 0.24 -> 5.46 mm
- net Net-(U1-USB_DM): track 0.00 -> 4.57 mm
- net XOUT: track 0.00 -> 4.48 mm
- net Net-(U1-USB_DP): track 0.00 -> 4.06 mm
- net XIN: track 0.00 -> 3.40 mm
- net SWCLK: track 20.0 -> 22.4 mm
- net Net-(J1-CC1): track 0.00 -> 2.26 mm
- net GPIO0: track 28.0 -> 26.0 mm
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- added copper zone on B.Cu, net GND
Other:
- board size 21.9 x 52.6 mm -> 22 x 54 mm

Commit message: copper pours
Parts:
- moved C17 1.05 mm to (98.0, 45.0)
- moved C15 0.66 mm to (94.2, 60.7)
Routing:
- net GPIO20: track 12.5 -> 10.8 mm
- net GPIO18: track 16.8 -> 15.3 mm
- net GPIO21: track 11.1 -> 9.67 mm
- net GPIO12: track 13.4 -> 12.2 mm
- net GPIO17: track 23.1 -> 22.2 mm
- net GPIO11: track 10.6 -> 10.0 mm
- net GPIO10: track 8.77 -> 8.26 mm
- net GND: track 0.00 -> 0.49 mm, vias 13 -> 6
- net (no net): vias 3 -> 1
- added copper zone on F.Cu, net GND
