File: _restore_backup_2026-09-15T12-37-06-078/rp2040_devboard.kicad_pcb (KiCad board)
At the start: 2 copper layers, 22 x 54 mm, 33 parts, among them J1 USB_C_Receptacle_USB2.0_14P, J2 Conn_01x20, J3 Conn_01x20, J4 Conn_01x03, SW1 SW_Push, U1 RP2040, U2 MCP1700x-330xxMB, U3 W25Q128JVS, Y1 Crystal_GND24

Commit message: fixed like 10 drc errors
Parts:
- moved R5 2.90 mm to (99.5, 59.6)
- moved C4 1.23 mm to (101.5, 55.4)
- moved C15 1.19 mm to (94.2, 60.7)
- moved R2 1.12 mm to (94.5, 35.5), turned to 180 degrees
- moved C13 0.95 mm to (99.8, 66.2)
- moved C16 0.85 mm to (97.5, 63.4)
- moved Y1 0.85 mm to (96.5, 60.8)
- moved R1 0.50 mm to (99.5, 35.5)
Routing:
- net VBUS: track 62.0 -> 22.1 mm, vias 2 -> 0
- net +3V3: track 84.4 -> 48.2 mm, vias 7 -> 0
- net USB_D-: track 17.0 -> 2.74 mm, vias 2 -> 0
- net RUN: track 10.7 -> 0.00 mm, vias 1 -> 0
- net GND: track 10.0 -> 0.49 mm, vias 12 -> 6
- net XOUT: track 6.79 -> 4.48 mm
- net Net-(C16-Pad1): track 3.36 -> 5.46 mm
- net XIN: track 5.36 -> 3.72 mm
- net GPIO29_ADC3: track 26.2 -> 24.6 mm
- net GPIO14: track 20.7 -> 19.9 mm
- net GPIO10: track 8.84 -> 8.26 mm
- net Net-(J1-CC1): track 2.76 -> 2.26 mm
